File: kicad/kicad-weight-scale-6-ch/kicad-weight-scale-6-ch.kicad_pcb (KiCad board)
At the start: 2 copper layers, 100 x 100 mm, 45 parts, among them J1 Barrel_Jack_Switch, J2 Conn_01x02, J3 Conn_01x04, J4 Conn_01x04, J5 Conn_01x04, J6 Conn_01x02, J7 Conn_01x02, J8 Conn_01x02, J9 Conn_01x02, Q1 Si4542DY, Q2 Si4542DY, Q3 AO3401A, SW1 SW_Push, U1 TP-4056, U10 USB_Type_C, U11 USB_Type_C, U12 USB_Type_C, U13 USB_Type_C, U2 StepUpTo5V, U3 WCMCU-ADS1232, U4 ESPWROOM32, U5 WCMCU-ADS1232, U6 DataLoggingBoard, U7 WCMCU-ADS1232, U8 USB_Type_C, U9 USB_Type_C

Commit message: Update nextion-esp32dws6chwl_ench.HMI, kicad-weight-scale-6-ch-cache.lib, and 6 more files...
Parts:
- removed G***: LOGO, myLogo:keyworks_logo
- Q3: value AO3401A -> BSS138
