File: kicad/kicad-weight-scale-6-ch/kicad-weight-scale-6-ch.kicad_pcb (KiCad board)
At the start: 2 copper layers, 100 x 100 mm, 44 parts, among them J1 Barrel_Jack_Switch, J2 Conn_01x02, J3 Conn_01x04, J4 Conn_01x04, J5 Conn_01x04, J6 Conn_01x02, J7 Conn_01x02, J8 Conn_01x02, J9 Conn_01x02, Q1 Si4542DY, Q2 Si4542DY, Q3 BSS138, SW1 SW_Push, U1 TP-4056, U10 USB_Type_C, U11 USB_Type_C, U12 USB_Type_C, U13 USB_Type_C, U2 StepUpTo5V, U3 WCMCU-ADS1232, U4 ESPWROOM32, U5 WCMCU-ADS1232, U6 DataLoggingBoard, U7 WCMCU-ADS1232, U8 USB_Type_C, U9 USB_Type_C

Commit message: Update nextion-esp32dws6chwl_ench.HMI, kicad-weight-scale-6-ch.kicad_pcb, and 20 more files...
Connections:
- Q2 pad 1: VCC_B1 -> (no net)
- Q2 pad 2: 5V -> (no net)
- Q2 pad 3: (no net) -> VCC_B1
- Q2 pad 4: (no net) -> 5V
- Q2 pad 5: (no net) -> Net-(D1-Pad2)
- Q2 pad 6: (no net) -> Net-(D1-Pad2)
- Q2 pad 7: Net-(D1-Pad2) -> (no net)
- Q2 pad 8: Net-(D1-Pad2) -> (no net)
Routing:
- net VCC_B1: track 15.2 -> 22.2 mm
- net 5V: track 28.0 -> 33.2 mm
- net Net-(D1-Pad2): track 8.06 -> 11.3 mm
