File: kicad/kicad-weight-scale-6-ch/kicad-weight-scale-6-ch.sch (KiCad schematic (older format))
At the start: 38 parts

Commit message: update PCB deisgn
Parts:
- removed J? (x6): Conn_01x04, symbol Connector_Generic:Conn_01x04
- removed Q?: Si4542DY, Package_SO:SOIC-8_3.9x4.9mm_P1.27mm, symbol Transistor_FET:Si4542DY
- removed U?: StepUpDC5V, symbol Step~Up~DC~to~5V~USB:StepUpDC5V
- removed U?: TP4056, symbol TP4056:TP4056
- removed U?: ESPWROOM32, symbol ESP~WROOM32~DEV-BOARD:ESPWROOM32
- added J1: Barrel_Jack_Switch, Connector_BarrelJack:BarrelJack_Horizontal, symbol Connector:Barrel_Jack_Switch
- added J3, J4, J5: Conn_01x04, Connector_PinHeader_2.54mm:PinHeader_1x04_P2.54mm_Vertical, symbol Connector_Generic:Conn_01x04
- added J9: Conn_01x02, Connector_PinHeader_2.54mm:PinHeader_1x02_P2.54mm_Vertical, symbol Connector_Generic:Conn_01x02
- added Q2: Si4542DY, Package_SO:SOIC-8_3.9x4.9mm_P1.27mm, symbol Transistor_FET:Si4542DY
- added R1, R3: 10k, Resistor_SMD:R_0805_2012Metric_Pad1.20x1.40mm_HandSolder, symbol Device:R
- added U1: TP-4056, DIY-Board:Li-ion ic charger, symbol TP4056:TP-4056
- added U10, U11, U12, U13, U8, U9: USB_Type_C, DIY-Board:Type C Converter, symbol USB~Type~C~Converter:USB_Type_C
- added U2: StepUpTo5V, DIY-Board:Step up 5V, symbol Step~Up~DC~to~5V~USB:StepUpTo5V
- added U4: ESPWROOM32, DIY-Board:esp wroom 32 board, symbol ESP~WROOM32~DEV-BOARD:ESPWROOM32
- BT1: footprint (none) -> TerminalBlock:TerminalBlock_bornier-2_P5.08mm
- BZ1: footprint (none) -> Buzzer_Beeper:Buzzer_12x9.5RM7.6
- C1, C2: renamed from C?; footprint (none) -> Capacitor_THT:CP_Radial_D7.5mm_P2.50mm
- D1, D2, D3: renamed from D?; footprint (none) -> Diode_SMD:D_SMA-SMB_Universal_Handsoldering
- J2, J6, J7, J8: renamed from J?; footprint (none) -> Connector_PinHeader_2.54mm:PinHeader_1x02_P2.54mm_Vertical
- R10, R11, R2, R4, R5, R6, R7, R8, R9: renamed from R?; footprint (none) -> Resistor_SMD:R_0805_2012Metric_Pad1.20x1.40mm_HandSolder
- SW1: renamed from SW?; footprint (none) -> Connector_PinHeader_2.54mm:PinHeader_1x02_P2.54mm_Vertical
- U3, U5, U7: renamed from U?; footprint (none) -> DIY-Board:wcmcu-ads1232
- U6: renamed from U?; footprint (none) -> DIY-Board:Datalogging board
- gave numbers to parts that had none: 2
Connections:
- net labels added: RXD0, RXD1, RXD2, SCLK_2, SPEED, TXD0, TXD1, TXD2
- wire segments 70 -> 75
Other:
- moved on the sheet: BT1, BZ1, C1, C2, D1, D2, D3, J2, J6, J7, J8, Q1A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

Commit message: Update nextion-esp32dws6chwl_ench.HMI, kicad-weight-scale-6-ch-cache.lib, and 6 more files...
Parts:
- removed Q3: AO3401A, Package_TO_SOT_SMD:SOT-23, symbol Transistor_FET:AO3401A
- added Q3: BSS138, Package_TO_SOT_SMD:SOT-23, symbol Transistor_FET:BSS138
Changed lines of the file:
@@
-$EndComp
-$Comp
-L Transistor_FET:AO3401A Q3
-U 1 1 606F53CC
-P 3800 6700
-F 0 "Q3" H 4005 6746 50  0000 L CNN
-F 1 "AO3401A" H 4005 6655 50  0000 L CNN
-F 2 "Package_TO_SOT_SMD:SOT-23" H 4000 6625 50  0001 L CIN
-F 3 "http://www.aosmd.com/pdfs/datasheet/AO3401A.pdf" H 3800 6700 50  0001 L CNN
-	1    3800 6700
-	1    0    0    -1
 $EndComp
 $Comp
@@
 	2540 1650 2750 1650
 Connection ~ 2540 2030
+$Comp
+L Transistor_FET:BSS138 Q3
+U 1 1 60917343
+P 3800 6700
+F 0 "Q3" H 4004 6746 50  0000 L CNN
+F 1 "BSS138" H 4004 6655 50  0000 L CNN
+F 2 "Package_TO_SOT_SMD:SOT-23" H 4000 6625 50  0001 L CIN
+F 3 "https://www.onsemi.com/pub/Collateral/BSS138-D.PDF" H 3800 6700 50  0001 L CNN
+	1    3800 6700
+	1    0    0    -1
+$EndComp
 $EndSCHEMATC
